File: lickport_array_module.kicad_pcb (KiCad board)
At the start: 2 copper layers, 203.2 x 147.3 mm, 189 parts, among them P1 PWR_JACK_2.5x5.5_SMD_VERT, P10 RECEPTACLE_2MM, P11 RECEPTACLE_2MM, P12 RECEPTACLE_2MM, P13 RECEPTACLE_2MM, P14 RECEPTACLE_2MM, P2 BNC, P3 RECEPTACLE_2MM, P4 RECEPTACLE_2MM, P5 RECEPTACLE_2MM, P6 RECEPTACLE_2MM, P7 RECEPTACLE_2MM, P8 RECEPTACLE_2MM, P9 RECEPTACLE_2MM, T1 TERM_BLK_ANG_2_PIN_3.5MM_PITCH, T10 TERM_BLK_ANG_2_PIN_3.5MM_PITCH, T11 TERM_BLK_ANG_2_PIN_3.5MM_PITCH, T12 TERM_BLK_ANG_2_PIN_3.5MM_PITCH, T2 TERM_BLK_ANG_2_PIN_3.5MM_PITCH, T3 TERM_BLK_ANG_2_PIN_3.5MM_PITCH, T4 TERM_BLK_ANG_2_PIN_3.5MM_PITCH, T5 TERM_BLK_ANG_2_PIN_3.5MM_PITCH, T6 TERM_BLK_ANG_2_PIN_3.5MM_PITCH, T7 TERM_BLK_ANG_2_PIN_3.5MM_PITCH, T8 TERM_BLK_ANG_2_PIN_3.5MM_PITCH, T9 TERM_BLK_ANG_2_PIN_3.5MM_PITCH, U1 AT42QT2120-MMHR, U10 DRV103, U11 DRV103, U12 DRV103, U13 DRV103, U2 DRV103, U3 DRV103, U4 DRV103, U5 DRV103, U6 DRV103, U7 DRV103, U8 DRV103, U9 DRV103

Commit message: Modify net classes
Connections:
- net Net-(R5-Pad2) renamed /RESET
Other:
- net class HIGHPOWER removed
- net class POWER: via_dia 0.8128 -> 0.6096
- net class SENSE: via_dia 0.9144 -> 1.0668
- net class SIGNAL: via_dia 0.8128 -> 0.6096
- net class THICKPOWER added: clearance 0.2032, trace_width 0.6096, via_dia 0.9144, via_drill 0.4064
- net class THICKSIGNAL added: clearance 0.2032, trace_width 0.6096, via_dia 0.9144, via_drill 0.4064

Commit message: Final layout before exporting files
Routing:
- net GND: track 0.00 -> 931.1 mm, vias 0 -> 2
- net VCC: track 0.00 -> 869.5 mm
- net /SOLENOID_4: track 0.00 -> 152.0 mm, vias 0 -> 1
- net /SOLENOID_1: track 0.00 -> 146.5 mm, vias 0 -> 1
- net /SOLENOID_3: track 0.00 -> 141.1 mm, vias 0 -> 1
- net /SYNC: track 0.00 -> 126.3 mm, vias 0 -> 1
- net /SOLENOID_0: track 0.00 -> 121.5 mm, vias 0 -> 2
- net /SOLENOID_10: track 0.00 -> 112.5 mm
- net /SOLENOID_7: track 0.00 -> 101.7 mm, vias 0 -> 1
- net /SOLENOID_5: track 0.00 -> 98.5 mm, vias 0 -> 1
- net /SOLENOID_2: track 0.00 -> 91.6 mm, vias 0 -> 1
- net /SOLENOID_6: track 0.00 -> 87.6 mm
- net /~CHANGE: track 0.00 -> 84.3 mm, vias 0 -> 1
- net /SDA: track 0.00 -> 66.2 mm, vias 0 -> 2
- net VDD: track 0.00 -> 62.8 mm, vias 0 -> 2
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- added copper zone on B.Cu, net GND
- added copper zone on F.Cu, net GND
Other:
- board text added: "POWER"
- board text added: "SYNC"
